File: odin_d_pannel_prototype.kicad_pcb (KiCad board)
At the start: 2 copper layers, 108 parts, among them J1 Conn_01x03, Q4 Q_NPN_BEC, Q5 Q_NPN_BEC, T1 BT136S

Commit message: Added files for production run
Parts:
- removed the C1 at (143.5, 88.3)
- removed the C1 at (143.5, 62.5)
- removed the C1 at (102.3, 88.3)
- removed the C2 at (143.5, 86.0)
- removed the C2 at (143.5, 60.2)
- removed the C2 at (102.3, 86.0)
- removed the C3 at (143.5, 83.8)
- removed the C3 at (143.5, 58.0)
- removed the C3 at (102.3, 83.8)
- removed the C4 at (170.2, 102.8)
- removed the C4 at (170.2, 77.0)
- removed the C4 at (128.9, 102.8)
- removed the D1 at (139.8, 81.4)
- removed the D1 at (139.8, 55.6)
- removed the D1 at (98.5, 81.4)
- removed the D2 at (145.9, 81.4)
- removed the D2 at (145.9, 55.6)
- removed the D2 at (104.7, 81.4)
- removed the J1 at (152.4, 92.1)
- removed the J1 at (152.4, 66.3)
- removed the J1 at (111.1, 92.1)
- removed the J1 at (111.1, 66.3)
- removed the PH1 at (152.8, 94.0)
- removed the PH1 at (152.8, 68.2)
- removed the PH1 at (111.5, 94.0)
- removed the PH1 at (111.5, 68.2)
- removed PH2 (x3): Q_Photo_NPN_EC, Resistor_SMD:R_0805_2012Metric
- removed the PH3 at (152.7, 96.2)
- removed the PH3 at (152.7, 70.3)
- removed the PH3 at (111.5, 96.2)
- removed the Q4 at (169.2, 98.8)
- removed the Q4 at (169.2, 73.0)
- removed the Q4 at (127.9, 98.8)
- removed the Q5 at (164.9, 99.7)
- removed the Q5 at (164.9, 73.9)
- removed the Q5 at (123.7, 99.7)
- removed the R0 at (141.6, 103.5)
- removed the R0 at (141.6, 77.7)
- removed the R0 at (100.3, 103.5)
- removed the R0 at (100.3, 77.7)
- removed the R1 at (134.4, 102.0)
- removed the R1 at (134.4, 76.2)
- removed the R1 at (93.2, 102.0)
- removed the R1 at (93.2, 76.2)
- removed the R10 at (156.8, 89.4)
- removed the R10 at (156.8, 63.6)
- removed the R10 at (115.6, 89.4)
- removed the R2 at (138.6, 96.8)
- removed the R2 at (138.6, 71.0)
- removed the R2 at (97.4, 96.8)
- removed the R2 at (97.4, 71.0)
- removed the R3 at (134.4, 92.4)
- removed the R3 at (134.4, 66.6)
- removed the R3 at (93.1, 92.4)
- removed the R3 at (93.1, 66.6)
- removed the R4 at (138.6, 87.4)
- removed the R4 at (138.6, 61.6)
- removed the R4 at (97.4, 87.4)
- removed the R4 at (97.4, 61.6)
- removed the R5 at (134.4, 82.8)
- removed the R5 at (134.4, 57.0)
- removed the R5 at (93.2, 82.8)
- removed the R5 at (93.2, 57.0)
- removed the R6 at (150.4, 100.4)
- removed the R6 at (150.4, 74.6)
- removed the R6 at (109.2, 100.4)
- removed the R7 at (153.5, 101.3)
- removed the R7 at (153.5, 75.5)
- removed the R7 at (112.3, 101.3)
- removed the R8 at (156.0, 99.9)
- removed the R8 at (156.0, 74.1)
- removed the R8 at (114.8, 99.9)
- removed the R9 at (170.2, 94.8)
- removed the R9 at (170.2, 69.0)
- removed the R9 at (128.9, 94.8)
- removed the RV1 at (150.2, 87.1)
- removed the RV1 at (150.2, 61.3)
- removed the RV1 at (108.9, 87.1)
- removed the RV2 at (148.8, 89.1)
- removed the RV2 at (148.8, 63.3)
- removed the RV2 at (107.6, 89.1)
- removed the RV3 at (153.6, 87.0)
- removed the RV3 at (153.6, 61.2)
- removed the RV3 at (112.4, 87.0)
- removed the T1 at (164.9, 85.2)
- removed the T1 at (164.9, 59.4)
- removed the T1 at (123.7, 85.2)
- removed the T1 at (123.7, 59.4)
- added C1: 10uF, Capacitor_SMD:C_0805_2012Metric, F.Cu at (160.0, 84.2)
- added C1: 10uF, Capacitor_SMD:C_0805_2012Metric, F.Cu at (118.6, 84.2)
- added C1: 10uF, Capacitor_SMD:C_0805_2012Metric, F.Cu at (160.0, 58.3)
- added C2: 10uF, Capacitor_SMD:C_0805_2012Metric, F.Cu at (160.0, 81.9)
- added C2: 10uF, Capacitor_SMD:C_0805_2012Metric, F.Cu at (118.6, 81.9)
- added C2: 10uF, Capacitor_SMD:C_0805_2012Metric, F.Cu at (160.0, 56.0)
- added C3: 10uF, Capacitor_SMD:C_0805_2012Metric, F.Cu at (160.0, 79.7)
- added C3: 10uF, Capacitor_SMD:C_0805_2012Metric, F.Cu at (118.6, 79.7)
- added C3: 10uF, Capacitor_SMD:C_0805_2012Metric, F.Cu at (160.0, 53.8)
- added C4: 10uF, Capacitor_SMD:C_0805_2012Metric, F.Cu at (167.4, 97.6)
- added C4: 10uF, Capacitor_SMD:C_0805_2012Metric, F.Cu at (126.1, 97.6)
- added C4: 10uF, Capacitor_SMD:C_0805_2012Metric, F.Cu at (167.4, 71.7)
- added D1: 1N4007, Diode_SMD:D_SOD-123, F.Cu at (156.2, 77.3)
- added D1: 1N4007, Diode_SMD:D_SOD-123, F.Cu at (114.9, 77.3)
- added D1: 1N4007, Diode_SMD:D_SOD-123, F.Cu at (156.2, 51.4)
- added D2: 12V, Diode_SMD:D_SOD-123, F.Cu at (162.4, 77.3)
- added D2: 12V, Diode_SMD:D_SOD-123, F.Cu at (121.0, 77.3)
- added D2: 12V, Diode_SMD:D_SOD-123, F.Cu at (162.4, 51.4)
- added J1: Conn_01x03, custom:nema_3_pin_chinese, F.Cu at (168.8, 88.0)
- added J1: Conn_01x03, custom:nema_3_pin_chinese, F.Cu at (127.5, 88.0)
- added J1: Conn_01x03, custom:nema_3_pin_chinese, F.Cu at (168.8, 62.1)
- added J1: Conn_01x03, custom:nema_3_pin_chinese, F.Cu at (127.5, 62.1)
- added PH1: Q_Photo_NPN_EC, Resistor_SMD:R_0805_2012Metric, F.Cu at (169.2, 87.8)
- added PH1: Q_Photo_NPN_EC, Resistor_SMD:R_0805_2012Metric, F.Cu at (127.9, 87.8)
- added PH1: Q_Photo_NPN_EC, Resistor_SMD:R_0805_2012Metric, F.Cu at (169.2, 62.0)
- added PH3: Q_Photo_NPN_EC, Resistor_SMD:R_1206_3216Metric, F.Cu at (168.8, 90.7)
- added PH3: Q_Photo_NPN_EC, Resistor_SMD:R_1206_3216Metric, F.Cu at (127.4, 90.7)
- added PH3: Q_Photo_NPN_EC, Resistor_SMD:R_1206_3216Metric, F.Cu at (168.8, 64.8)
- added Q4: Q_NPN_BEC, Package_TO_SOT_SMD:SOT-23, F.Cu at (177.4, 97.3)
- added Q4: Q_NPN_BEC, Package_TO_SOT_SMD:SOT-23, F.Cu at (136.0, 97.3)
- added Q4: Q_NPN_BEC, Package_TO_SOT_SMD:SOT-23, F.Cu at (177.4, 71.4)
- added Q5: Q_NPN_BEC, Package_TO_SOT_SMD:SOT-23, F.Cu at (173.3, 95.3)
- added Q5: Q_NPN_BEC, Package_TO_SOT_SMD:SOT-23, F.Cu at (131.9, 95.3)
- added Q5: Q_NPN_BEC, Package_TO_SOT_SMD:SOT-23, F.Cu at (173.3, 69.4)
- added R0: 3k, Resistor_SMD:R_1210_3225Metric, F.Cu at (160.9, 98.6)
- added R0: 3k, Resistor_SMD:R_1210_3225Metric, F.Cu at (119.6, 98.6)
- added R0: 3k, Resistor_SMD:R_1210_3225Metric, F.Cu at (160.9, 72.7)
- added R0: 3k, Resistor_SMD:R_1210_3225Metric, F.Cu at (119.6, 72.7)
- added R1: 3k, Resistor_SMD:R_1210_3225Metric, F.Cu at (151.3, 97.9)
- added R1: 3k, Resistor_SMD:R_1210_3225Metric, F.Cu at (110.0, 97.9)
- added R1: 3k, Resistor_SMD:R_1210_3225Metric, F.Cu at (151.3, 72.0)
- added R1: 3k, Resistor_SMD:R_1210_3225Metric, F.Cu at (110.0, 72.0)
- added R10: 2.2k, Resistor_SMD:R_0805_2012Metric, F.Cu at (174.3, 86.4)
- added R10: 2.2k, Resistor_SMD:R_0805_2012Metric, F.Cu at (133.0, 86.4)
- added R10: 2.2k, Resistor_SMD:R_0805_2012Metric, F.Cu at (174.3, 60.5)
- added R2: 3k, Resistor_SMD:R_1210_3225Metric, F.Cu at (155.1, 92.7)
- added R2: 3k, Resistor_SMD:R_1210_3225Metric, F.Cu at (113.8, 92.7)
- added R2: 3k, Resistor_SMD:R_1210_3225Metric, F.Cu at (155.1, 66.8)
- added R2: 3k, Resistor_SMD:R_1210_3225Metric, F.Cu at (113.8, 66.8)
- added R3: 3k, Resistor_SMD:R_1210_3225Metric, F.Cu at (151.3, 88.3)
- added R3: 3k, Resistor_SMD:R_1210_3225Metric, F.Cu at (110.0, 88.3)
- added R3: 3k, Resistor_SMD:R_1210_3225Metric, F.Cu at (151.3, 62.4)
- added R3: 3k, Resistor_SMD:R_1210_3225Metric, F.Cu at (110.0, 62.4)
- added R4: 3k, Resistor_SMD:R_1210_3225Metric, F.Cu at (155.1, 83.3)
- added R4: 3k, Resistor_SMD:R_1210_3225Metric, F.Cu at (113.8, 83.3)
- added R4: 3k, Resistor_SMD:R_1210_3225Metric, F.Cu at (155.1, 57.4)
- added R4: 3k, Resistor_SMD:R_1210_3225Metric, F.Cu at (113.8, 57.4)
- added R5: 3k, Resistor_SMD:R_1210_3225Metric, F.Cu at (151.3, 78.7)
- added R5: 3k, Resistor_SMD:R_1210_3225Metric, F.Cu at (110.0, 78.7)
- added R5: 3k, Resistor_SMD:R_1210_3225Metric, F.Cu at (151.3, 52.8)
- added R5: 3k, Resistor_SMD:R_1210_3225Metric, F.Cu at (110.0, 52.8)
- added R6: 30k, Resistor_SMD:R_0805_2012Metric, F.Cu at (165.6, 87.9)
- added R6: 30k, Resistor_SMD:R_0805_2012Metric, F.Cu at (124.2, 87.9)
- added R6: 30k, Resistor_SMD:R_0805_2012Metric, F.Cu at (165.6, 62.0)
- added R7: 30k, Resistor_SMD:R_0805_2012Metric, F.Cu at (167.4, 94.1)
- added R7: 30k, Resistor_SMD:R_0805_2012Metric, F.Cu at (126.1, 94.1)
- added R7: 30k, Resistor_SMD:R_0805_2012Metric, F.Cu at (167.4, 68.2)
- added R8: 30k, Resistor_SMD:R_0805_2012Metric, F.Cu at (170.2, 94.1)
- added R8: 30k, Resistor_SMD:R_0805_2012Metric, F.Cu at (128.9, 94.1)
- added R8: 30k, Resistor_SMD:R_0805_2012Metric, F.Cu at (170.2, 68.2)
- added R9: 2.2k, Resistor_SMD:R_0805_2012Metric, F.Cu at (180.6, 97.2)
- added R9: 2.2k, Resistor_SMD:R_0805_2012Metric, F.Cu at (139.2, 97.2)
- added R9: 2.2k, Resistor_SMD:R_0805_2012Metric, F.Cu at (180.6, 71.3)
- added RV1: Varistor, Varistor:RV_Disc_D12mm_W4.3mm_P7.5mm, B.Cu at (166.6, 83.0)
- added RV1: Varistor, Varistor:RV_Disc_D12mm_W4.3mm_P7.5mm, B.Cu at (125.3, 83.0)
- added RV1: Varistor, Varistor:RV_Disc_D12mm_W4.3mm_P7.5mm, B.Cu at (166.6, 57.1)
- added RV2: Varistor, Varistor:RV_Disc_D9mm_W4.1mm_P5mm, B.Cu at (165.3, 85.0)
- added RV2: Varistor, Varistor:RV_Disc_D9mm_W4.1mm_P5mm, B.Cu at (124.0, 85.0)
- added RV2: Varistor, Varistor:RV_Disc_D9mm_W4.1mm_P5mm, B.Cu at (165.3, 59.1)
- added RV3: Varistor, Varistor:RV_Disc_D21.5mm_W5.8mm_P10mm, B.Cu at (170.1, 83.0)
- added RV3: Varistor, Varistor:RV_Disc_D21.5mm_W5.8mm_P10mm, B.Cu at (128.7, 83.0)
- added RV3: Varistor, Varistor:RV_Disc_D21.5mm_W5.8mm_P10mm, B.Cu at (170.1, 57.0)
- added T1: BT136S, Package_TO_SOT_SMD:TO-252-2, F.Cu at (183.0, 84.3)
- added T1: BT136S, Package_TO_SOT_SMD:TO-252-2, F.Cu at (141.7, 84.3)
- added T1: BT136S, Package_TO_SOT_SMD:TO-252-2, F.Cu at (183.0, 58.4)
- added T1: BT136S, Package_TO_SOT_SMD:TO-252-2, F.Cu at (141.7, 58.4)
- moved R6 19.6 mm to (124.2, 62.0)
- moved R10 17.7 mm to (133.0, 60.5), turned to 180 degrees
- moved PH1 16.9 mm to (127.9, 62.0)
- moved C1 16.9 mm to (118.6, 58.3)
- moved C2 16.9 mm to (118.6, 56.0)
- moved C3 16.9 mm to (118.6, 53.8)
- moved RV2 16.9 mm to (124.0, 59.1)
- moved RV3 16.9 mm to (128.7, 57.0)
- moved D1 16.9 mm to (114.9, 51.4)
- moved RV1 16.9 mm to (125.3, 57.1)
- moved D2 16.9 mm to (121.0, 51.4)
- moved PH3 16.9 mm to (127.4, 64.8)
- moved R7 15.6 mm to (126.1, 68.2)
- moved R8 15.3 mm to (128.9, 68.2)
- moved R9 10.6 mm to (139.2, 71.3), turned to 270 degrees
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- renumbered PH2 to PH1
Routing:
- net /GND: track 253.9 -> 121.5 mm
- net /NEUTRAL: track 32.6 -> 0.00 mm
- net Net-(Q5-Pad3): track 60.1 -> 34.5 mm
- net Net-(R0-Pad1): track 23.1 -> 0.00 mm
- net Net-(C4-Pad1): track 77.9 -> 55.8 mm
- net Net-(R1-Pad1): track 20.8 -> 0.00 mm
- net Net-(PH1-Pad1): track 45.1 -> 28.4 mm
- net Net-(Q4-Pad3): track 56.1 -> 41.1 mm
- net /LIVE: track 55.1 -> 45.5 mm
- net Net-(Q4-Pad2): track 33.3 -> 29.6 mm
- net Net-(R10-Pad1): track 17.5 -> 14.5 mm
- net /LOAD: track 0.00 -> 1.68 mm
